Commit message: finished unit 1

File: my_mira_description/urdf/mira.urdf (robot description, URDF)
Before this commit: robot mira, 2 links, 1 joints
Links:
- added link camera_link; visual box size=0.0005 0.0005 0.0005
- added link head_link; visual mesh filename=package://my_mira_description/models/mira/meshes/mira_head_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
- added link left_eye_link; visual mesh filename=package://my_mira_description/models/mira/meshes/mira_eye_v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
- added link pitch_M2_link; visual cylinder length=0.005 radius=0.01
- added link right_eye_link; visual mesh filename=package://my_mira_description/models/mira/meshes/mira_eye_v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
- added link yaw_M3_link; visual cylinder length=0.005 radius=0.01
- link base_link: geometry visual mesh filename=package://my_mira_description/models/mira/meshes/mira_body_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
- link roll_M1_link: geometry visual cylinder length=0.005 radius=0.01
Joints:
- added joint base_head_joint: type fixed, parent yaw_M3_link, child head_link, origin xyz=0 0 0 rpy=0 0 0
- added joint head_camera_joint: type fixed, parent head_link, child camera_link, origin xyz=0 0.057 0.0255 rpy=0 0 0
- added joint head_lefteye_joint: type fixed, parent head_link, child left_eye_link, origin xyz=0.0095 0.057 0.0085 rpy=-1.5708 0 0
- added joint head_righteye_joint: type fixed, parent head_link, child right_eye_link, origin xyz=-0.0095 0.057 0.0085 rpy=-1.5708 0 0
- added joint pitch_joint: type revolute, parent roll_M1_link, child pitch_M2_link, origin xyz=0 0 0 rpy=0 -1.5708 0, axis 0 1 0, limit lower=0 upper=0.44 effort=0.1 velocity=0.005
- added joint yaw_joint: type continuous, parent pitch_M2_link, child yaw_M3_link, origin xyz=0.01 0 rpy=0 1.5708 0, axis 0 0 1, limit effort=0.1 velocity=0.01

Commit message: added inertials and collisions, and got the basic shape representations to spawn in gazebo, but .dae mesh files refuse to spawn. Also, When i used <mesh $MODEL> instead of <mesh filename://> the inertials became extremely fucked up, and it started gaining momentum and started spinning around like a top (not in place)

File: my_mira_description/urdf/mira.urdf (robot description, URDF)
Before this commit: robot mira, 8 links, 7 joints
Links:
- link base_link: mass None -> 0.18; geometry collision cylinder length=0.09 radius=0.06; visual mesh model=package://my_mira_description/models/mira_body_v3.dae
- link camera_link: mass None -> 0.001
- link head_link: mass None -> 0.02; geometry collision sphere radius=0.06; visual sphere radius=0.06
- link left_eye_link: mass None -> 0.001
- link pitch_M2_link: mass None -> 0.001
- link right_eye_link: mass None -> 0.001; geometry visual cylinder length=0.00525 radius=0.00525
- link roll_M1_link: mass None -> 0.001
- link yaw_M3_link: mass None -> 0.001
Joints:
- joint yaw_joint: origin xyz=0.01 0 rpy=0 1.5708 0 -> xyz=0.01 0 0 rpy=0 1.5708 0

Commit message: restored my version of launch files

File: my_mira_description/urdf/mira.urdf (robot description, URDF)
Before this commit: robot mira, 8 links, 7 joints
Links:
- link base_link: geometry collision cylinder length=0.09 radius=0.06; visual mesh filename=package://my_mira_description/models/mira/meshes/mira_body_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
- link head_link: geometry collision sphere radius=0.06; visual mesh filename=package://my_mira_description/models/mira/meshes/mira_head_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

Commit message: issue with dae spawn was a server bug, RobotIgniteAcademy is fixing it as we speak. for the package, drop the <my> from <my_mira_description>  in the <mesh filename>, so <mesh filename=[package://mira_description/models...]>

File: my_mira_description/urdf/mira.urdf (robot description, URDF)
Before this commit: robot mira, 8 links, 7 joints
Links:
- link base_link: geometry collision cylinder length=0.09 radius=0.06; visual mesh filename=package://mira_description/models/mira/meshes/mira_body_v3.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
- link head_link: geometry collision sphere radius=0.06; visual mesh filename=package://mira_description/models/mira/meshes/mira_head_v5.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
- link left_eye_link: geometry visual mesh filename=package://mira_description/models/mira/meshes/mira_eye_v4.d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
- link right_eye_link: geometry visual mesh filename=package://mira_description/models/mira/meshes/mira_eye_v4.d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
