Commit message: finished rviz spawn, and added collisions and inertials. currently spawning in gazebo. spawning only the 3 ball feet seems normal, but spawning everything together, both upper and lower leg links fall under ground plane when gurdy spawns, and drops a little. next move might be to measure each joint and spawn each so that its perfectly in a standing pose

File: my_gurdy_description/urdf/gurdy.urdf (robot description, URDF)
Before this commit: robot gurdy, 2 links, 1 joints
Links:
- added link footM1_link, mass 0.01; collision sphere radius=0.008; visual sphere radius=0.008
- added link footM2_link, mass 0.01; collision sphere radius=0.008; visual sphere radius=0.008
- added link footM3_link, mass 0.01; collision sphere radius=0.008; visual sphere radius=0.008
- added link lowerleg_M1_link, mass 0.01; collision cylinder length=0.06 radius=0.0015; visual mesh filename=package://gurdy_description/models/gurdy/meshes/gurdy_lower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
- added link lowerleg_M2_link, mass 0.01; collision cylinder length=0.06 radius=0.0015; visual mesh filename=package://gurdy_description/models/gurdy/meshes/gurdy_lower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
- added link lowerleg_M3_link, mass 0.01; collision cylinder length=0.06 radius=0.0015; visual mesh filename=package://gurdy_description/models/gurdy/meshes/gurdy_lower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
- added link upperleg_M1_link, mass 0.01; collision cylinder length=0.06 radius=0.0025; visual mesh filename=package://gurdy_description/models/gurdy/meshes/gurdy_highe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
- added link upperleg_M2_link, mass 0.01; collision cylinder length=0.06 radius=0.0025; visual mesh filename=package://gurdy_description/models/gurdy/meshes/gurdy_highe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
- added link upperleg_M3_link, mass 0.01; collision cylinder length=0.06 radius=0.0025; visual mesh filename=package://gurdy_description/models/gurdy/meshes/gurdy_highe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
- link base_link: mass None -> 0.001
- link head_link: mass None -> 0.01; geometry collision mesh filename=package://gurdy_description/models/gurdy/meshes/gurdy_head_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; visual mesh filename=package://gurdy_description/models/gurdy/meshes/gurdy_head_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
Joints:
- added joint basefoot_peg_M1_basefoot_peg_M1_joint_joint: type fixed, parent lowerleg_M1_link, child footM1_link, origin xyz=0 0 0.06 rpy=0 0 0
- added joint basefoot_peg_M2_basefoot_peg_M2_joint_joint: type fixed, parent lowerleg_M2_link, child footM2_link, origin xyz=0 0 0.06 rpy=0 0 0
- added joint basefoot_peg_M3_basefoot_peg_M3_joint_joint: type fixed, parent lowerleg_M3_link, child footM3_link, origin xyz=0 0 0.06 rpy=0 0 0
- added joint head_upperlegM1_joint: type revolute, parent head_link, child upperleg_M1_link, origin xyz=-0.02165 -0.0125 -0.008 rpy=3.14159 -1.05879e-22 0.523599, axis 0 1 0, limit lower=-1.57 upper=-0.1 effort=1.0 velocity=0.005
- added joint head_upperlegM2_joint: type revolute, parent head_link, child upperleg_M2_link, origin xyz=0.02165 -0.0125 -0.008 rpy=3.14159 0 2.61799, axis 0 1 0, limit lower=-1.57 upper=-0.1 effort=1.0 velocity=0.005
- added joint head_upperlegM3_joint: type revolute, parent head_link, child upperleg_M3_link, origin xyz=0 0.025 -0.008 rpy=3.14159 0 -1.5708, axis 0 1 0, limit lower=-1.57 upper=-0.1 effort=1.0 velocity=0.005
- added joint upperlegM1_lowerlegM1_joint: type revolute, parent upperleg_M1_link, child lowerleg_M1_link, origin xyz=0 0.0095 0.06 rpy=0 0 3.14159, axis 0 1 0, limit lower=-2.65 upper=0 effort=1.0 velocity=0.005
- added joint upperlegM2_lowerlegM2_joint: type revolute, parent upperleg_M2_link, child lowerleg_M2_link, origin xyz=0 0.0095 0.06 rpy=0 0 3.14159, axis 0 1 0, limit lower=-2.65 upper=0 effort=1.0 velocity=0.005
- added joint upperlegM3_lowerlegM3_joint: type revolute, parent upperleg_M3_link, child lowerleg_M3_link, origin xyz=0 0.0095 0.06 rpy=0 0 3.14159, axis 0 1 0, limit lower=-2.65 upper=0 effort=1.0 velocity=0.005

Commit message: simulated solution code, but has same problems of feet being under ground plane as my code

File: my_gurdy_description/urdf/gurdy.urdf (robot description, URDF)
Before this commit: robot gurdy, 11 links, 10 joints
Links:
- link base_link: mass 0.001 -> None; geometry collision box size=0.01 0.01 0.01; visual box size=0.01 0.01 0.01
- link head_link: geometry collision cylinder length=0.04 radius=0.05; visual mesh filename=package://gurdy_description/models/gurdy/meshes/gurdy_head_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
Joints:
- removed joint base_head_joint
- added joint fixed: type fixed, parent base_link, child head_link
- joint head_upperlegM1_joint: limit lower=-1.57 upper=-0.1 effort=1.0 velocity=0.005 -> lower=-1.55 upper=0.0 effort=1.0 velocity=0.005; origin xyz=-0.02165 -0.0125 -0.008 rpy=3.14159 -1.05879e-22 0.523599 -> xyz=-0.02165 -0.0125 -0.008 rpy=3.14159 0 0.523599
- joint head_upperlegM2_joint: limit lower=-1.57 upper=-0.1 effort=1.0 velocity=0.005 -> lower=-1.55 upper=0.0 effort=1.0 velocity=0.005
- joint head_upperlegM3_joint: limit lower=-1.57 upper=-0.1 effort=1.0 velocity=0.005 -> lower=-1.55 upper=0.0 effort=1.0 velocity=0.005
- joint upperlegM1_lowerlegM1_joint: limit lower=-2.65 upper=0 effort=1.0 velocity=0.005 -> lower=-2.9 upper=1.5708 effort=1.0 velocity=0.005; type revolute -> continuous
- joint upperlegM2_lowerlegM2_joint: limit lower=-2.65 upper=0 effort=1.0 velocity=0.005 -> lower=-2.9 upper=1.5708 effort=1.0 velocity=0.005
- joint upperlegM3_lowerlegM3_joint: limit lower=-2.65 upper=0 effort=1.0 velocity=0.005 -> lower=-2.9 upper=1.5708 effort=1.0 velocity=0.005

Commit message: added transmissions

File: my_gurdy_description/urdf/gurdy.urdf (robot description, URDF)
Before this commit: robot gurdy, 11 links, 10 joints
Joints:
- removed joint fixed
- added joint base_head_joint: type fixed, parent base_link, child head_link
- joint head_upperlegM1_joint: limit lower=-1.55 upper=0.0 effort=1.0 velocity=0.005 -> lower=-1.57 upper=0.0 effort=1.0 velocity=0.005; origin xyz=-0.02165 -0.0125 -0.008 rpy=3.14159 0 0.523599 -> xyz=-0.02165 -0.0125 -0.008 rpy=3.14159 -1.05879e-22 0.523599
- joint head_upperlegM2_joint: limit lower=-1.55 upper=0.0 effort=1.0 velocity=0.005 -> lower=-1.57 upper=0.0 effort=1.0 velocity=0.005
- joint head_upperlegM3_joint: limit lower=-1.55 upper=0.0 effort=1.0 velocity=0.005 -> lower=-1.57 upper=0.0 effort=1.0 velocity=0.005
- joint upperlegM1_lowerlegM1_joint: limit lower=-2.9 upper=1.5708 effort=1.0 velocity=0.005 -> lower=-2.65 upper=0 effort=1.0 velocity=0.005; type continuous -> revolute
- joint upperlegM2_lowerlegM2_joint: limit lower=-2.9 upper=1.5708 effort=1.0 velocity=0.005 -> lower=-2.65 upper=0 effort=1.0 velocity=0.005
- joint upperlegM3_lowerlegM3_joint: limit lower=-2.9 upper=1.5708 effort=1.0 velocity=0.005 -> lower=-2.65 upper=0 effort=1.0 velocity=0.005

Commit message: finished unit 4, creating gurdy from scratch!

File: my_gurdy_description/urdf/gurdy.urdf (robot description, URDF)
Before this commit: robot gurdy, 11 links, 10 joints
Joints:
- joint head_upperlegM1_joint: origin xyz=-0.02165 -0.0125 -0.008 rpy=3.14159 -1.05879e-22 0.523599 -> xyz=-0.02165 -0.0125 -0.008 rpy=3.14159 0 0.523599
