Commit message: XACROS are amazing!!! Did the examples up until parameterised macros. continue there, then XACRify completely gurdy.urdf

File: my_gurdy_description/robots/gurdy.urdf.xacro (robot description, xacro)
@@ -1,6 +1,5 @@
 <?xml version="1.0"?>
-<robot name="gurdy">
-<!--rosservice call /gazebo/delete_model "model_name: 'mira'"-->
-<!--roslaunch my_mira_description spawn_mira.launch-->
+<!-- <robot name="gurdy"> -->
+<robot xmlns:xacro="http://www.ros.org/wiki/xacro" name="gurdy">
 <!--You will also need the dimensions of the the basic geometry to have some idea of the way that everything is connected, and the collision elements geometry:-->
 <!--For base_link there is no inertia needed because its a non-functional element-->
@@ -17,4 +16,40 @@
 <!--PID are tricky. Use rqt_reconfigure to get correct values. These are some orientative values:-->
 <!--{p: 3.0, i: 1.0, d: 0.0}-->
+<!-- ################### XACRO Definitions ############################# -->
+<!-- ################### XACRO Definitions ############################# -->
+<!-- ################### XACRO Definitions ############################# -->
+<!-- ################### XACRO Definitions ############################# -->
+<!-- ################### XACRO Definitions ############################# -->
+<!-- MUST ALWAYS GO BEFORE XACRO DEFINITIONS -->
+<gazebo>
+    <plugin name="gazebo_ros_control" filename="libgazebo_ros_control.so">
+        <robotNamespace>/gurdy</robotNamespace>
+    </plugin>
+</gazebo>
+<xacro:property name="m" value="0.01"/>
+<xacro:property name="head_radius" value="0.05"/>
+<xacro:property name="head_length" value="0.04"/>
+<xacro:property name="head_z_origin" value="0.02"/>
+<xacro:property name="upperleg_M1_z_origin" value="0.02"/>
+<xacro:property name="upperleg_radius" value="0.0025"/>
+<xacro:property name="upperleg_length" value="0.06"/>
+<!-- You can perform the basic operations (+,-,*,/), the unary minus, and use parenthesis. This allows you to, for example, calculate the inertias based on the dimensions directly in the XACRO file. -->
+<xacro:property name="head_ixx" value="${( (m/12.0) * (3*head_radius*head_radius + head_length*head_length) )}"/>
+<!-- Another example would be symmetrically-positioned links or joints. -->
+<xacro:property name="head_iyy" value="${head_ixx}"/>
+<xacro:property name="head_izz" value="( (m*head_radius*head_radius) / (2.0) )"/>
+<!-- MACROS
+This is by far the most useful feature of XACROS. There are two main types of MACROS: -->
+<!-- SIMPLE MACRO -->
+<xacro:macro name="default_origin">
+    <origin xyz="0 0 0" rpy="0 0 0"/>
+</xacro:macro>
+<xacro:macro name="visual_origin">
+    <xacro:default_origin/>
+</xacro:macro>
+<!-- PARAMETERISED MACRO -->
+<xacro:property name="" value=""/>
+<xacro:property name="" value=""/>
+<xacro:property name="" value=""/>
 <!-- ################### LINK Definitions ############################# -->
 <!-- ################### LINK Definitions ############################# -->
@@ -29,5 +64,5 @@
         <!--</inertial>-->
         <collision>
-            <origin xyz="0 0 0" rpy="0 0 0"/>
+            <xacro:default_origin/>
             <geometry>
                 <box size="0.01 0.01 0.01"/>
@@ -35,5 +70,5 @@
         </collision>
         <visual>
-            <origin xyz="0 0 0" rpy="0 0 0"/>
+            <xacro:visual_origin/>
             <geometry>
                 <box size="0.01 0.01 0.01"/>
@@ -43,17 +78,18 @@
             <link name="head_link">
                 <inertial>
-                    <origin xyz="0 0 0.02" rpy="0 0 0"/>
-                    <mass value="0.01"/>
-                    <inertia ixx="7.58333333333e-06" ixy="0.0" ixz="0.0" iyy="7.58333333333e-06" iyz="0.0" izz="1.25e-05"/>
+                    <origin xyz="0 0 ${head_z_origin}" rpy="0 0 0"/>
+                    <mass value="${m}"/>
+                    <!-- <inertia ixx="7.58333333333e-06" ixy="0.0" ixz="0.0" iyy="7.58333333333e-06" iyz="0.0" izz="1.25e-05"/> -->
+                    <inertia ixx="${head_ixx}" ixy="0.0" ixz="0.0" iyy="head_iyy" iyz="0.0" izz="head_izz"/>
                 </inertial>
                 <collision>
-                    <origin xyz="0 0 0.02" rpy="0 0 0"/>
+                    <origin xyz="0 0 ${head_z_origin}" rpy="0 0 0"/>
                     <geometry>
-                        <cylinder radius="0.05" length="0.04"/>
+                        <cylinder radius="${head_radius}" length="${head_length}"/>
                         <!-- <mesh filename="package://gurdy_description/models/gurdy/meshes/gurdy_head_v2.dae"/> -->
                     </geometry>
                 </collision>
                 <visual>
-                    <origin xyz="0 0 0" rpy="0 0 0"/>
+                    <xacro:visual_origin/>
                     <geometry>
                         <mesh filename="package://gurdy_description/models/gurdy/meshes/gurdy_head_v2.dae"/>
@@ -63,6 +99,6 @@
                     <link name="upperleg_M1_link">
                         <inertial>
-                            <origin xyz="0 0 0.03" rpy="0 0 0"/> <!--UPPER-->
-                            <mass value="0.01"/>
+                            <origin xyz="0 0 ${upperleg_M1_z_origin}" rpy="0 0 0"/> <!--UPPER-->
+                            <mass value="${m}"/>
                             <!-- ORIGINAL value taken from Inertial_calculator.py -->
                             <!-- <inertia ixx="3.015625e-06" ixy="0.0" ixz="0.0" iyy="3.015625e-06" iyz="0.0" izz="3.125e-08"/> -->
@@ -71,11 +107,11 @@
                         </inertial>
                         <collision>
-                            <origin xyz="0 0 0.03" rpy="0 0 0"/> <!--UPPER COLLISION-->
+                            <origin xyz="0 0 ${upperleg_M1_z_origin}" rpy="0 0 0"/> <!--UPPER COLLISION-->
                             <geometry>
-                                <cylinder radius="0.0025" length="0.06"/>
+                                <cylinder radius="${upperleg_radius}" length="${upperleg_length}"/>
                             </geometry>
                         </collision>
                         <visual>
-                            <origin xyz="0 0 0" rpy="0 0 0"/>
+                            <xacro:visual_origin/>
                             <geometry>
                                 <mesh filename="package://gurdy_description/models/gurdy/meshes/gurdy_higherleg_v2.dae"/>
@@ -85,6 +121,6 @@
                     <link name="upperleg_M2_link">
                         <inertial>
-                            <origin xyz="0 0 0.03" rpy="0 0 0"/> <!--UPPER-->
-                            <mass value="0.01"/>
+                            <origin xyz="0 0 ${upperleg_M1_z_origin}" rpy="0 0 0"/> <!--UPPER-->
+                            <mass value="${m}"/>
                             <!-- ORIGINAL value taken from Inertial_calculator.py -->
                             <!-- <inertia ixx="3.015625e-06" ixy="0.0" ixz="0.0" iyy="3.015625e-06" iyz="0.0" izz="3.125e-08"/> -->
@@ -93,11 +129,11 @@
                         </inertial>
                         <collision>
-                            <origin xyz="0 0 0.03" rpy="0 0 0"/> <!--UPPER COLLISION-->
+                            <origin xyz="0 0 ${upperleg_M1_z_origin}" rpy="0 0 0"/> <!--UPPER COLLISION-->
                             <geometry>
-                                <cylinder radius="0.0025" length="0.06"/>
+                                <cylinder radius="${upperleg_radius}" length="${upperleg_length}"/>
                             </geometry>
                         </collision>
                         <visual>
-                            <origin xyz="0 0 0" rpy="0 0 0"/>
+                            <xacro:visual_origin/>
                             <geometry>
                                 <mesh filename="package://gurdy_description/models/gurdy/meshes/gurdy_higherleg_v2.dae"/>
@@ -107,6 +143,6 @@
                     <link name="upperleg_M3_link">
                         <inertial>
-                            <origin xyz="0 0 0.03" rpy="0 0 0"/> <!--UPPER-->
-                            <mass value="0.01"/>
+                            <origin xyz="0 0 ${upperleg_M1_z_origin}" rpy="0 0 0"/> <!--UPPER-->
+                            <mass value="${m}"/>
                             <!-- ORIGINAL value taken from Inertial_calculator.py -->
                             <!-- <inertia ixx="3.015625e-06" ixy="0.0" ixz="0.0" iyy="3.015625e-06" iyz="0.0" izz="3.125e-08"/> -->
@@ -115,11 +151,11 @@
                         </inertial>
                         <collision>
-                            <origin xyz="0 0 0.03" rpy="0 0 0"/> <!--UPPER COLLISION-->
+                            <origin xyz="0 0 ${upperleg_M1_z_origin}" rpy="0 0 0"/> <!--UPPER COLLISION-->
                             <geometry>
-                                <cylinder radius="0.0025" length="0.06"/>
+                                <cylinder radius="${upperleg_radius}" length="${upperleg_length}"/>
                             </geometry>
                         </collision>
                         <visual>
-                            <origin xyz="0 0 0" rpy="0 0 0"/>
+                            <xacro:visual_origin/>
                             <geometry>
                                 <mesh filename="package://gurdy_description/models/gurdy/meshes/gurdy_higherleg_v2.dae"/>
@@ -130,5 +166,5 @@
                                 <inertial>
                                     <origin xyz="0 0 0.03" rpy="0 0 0"/> <!--LOWER-->
-                                    <mass value="0.01"/>
+                                    <mass value="${m}"/>
                                     <!-- ORIGINAL value taken from Inertial_calculator.py -->
                                     <!-- <inertia ixx="3.005625e-06" ixy="0.0" ixz="0.0" iyy="3.005625e-06" iyz="0.0" izz="1.125e-08"/> -->
@@ -143,5 +179,5 @@
                                 </collision>
                                 <visual>
-                                    <origin xyz="0 0 0" rpy="0 0 0"/>
+                                    <xacro:visual_origin/>
                                     <geometry>
                                         <mesh filename="package://gurdy_description/models/gurdy/meshes/gurdy_lowerleg_v2.dae"/>
@@ -152,5 +188,5 @@
                                 <inertial>
                                     <origin xyz="0 0 0.03" rpy="0 0 0"/> <!--LOWER-->
-                                    <mass value="0.01"/>
+                                    <mass value="${m}"/>
                                     <!-- ORIGINAL value taken from Inertial_calculator.py -->
                                     <!-- <inertia ixx="3.005625e-06" ixy="0.0" ixz="0.0" iyy="3.005625e-06" iyz="0.0" izz="1.125e-08"/> -->
@@ -165,5 +201,5 @@
                                 </collision>
                                 <visual>
-                                    <origin xyz="0 0 0" rpy="0 0 0"/>
+                                    <xacro:visual_origin/>
                                     <geometry>
                                         <mesh filename="package://gurdy_description/models/gurdy/meshes/gurdy_lowerleg_v2.dae"/>
@@ -174,5 +210,5 @@
                                 <inertial>
                                     <origin xyz="0 0 0.03" rpy="0 0 0"/> <!--LOWER-->
-                                    <mass value="0.01"/>
+                                    <mass value="${m}"/>
                                     <!-- ORIGINAL value taken from Inertial_calculator.py -->
                                     <!-- <inertia ixx="3.005625e-06" ixy="0.0" ixz="0.0" iyy="3.005625e-06" iyz="0.0" izz="1.125e-08"/> -->
@@ -187,5 +223,5 @@
                                 </collision>
                                 <visual>
-                                    <origin xyz="0 0 0" rpy="0 0 0"/>
+                                    <xacro:visual_origin/>
                                     <geometry>
                                         <mesh filename="package://gurdy_description/models/gurdy/meshes/gurdy_lowerleg_v2.dae"/>
@@ -196,5 +232,5 @@
                                         <inertial>
                                             <origin xyz="0 0 0.01" rpy="0 0 0"/> <!--FOOT-->
-                                            <mass value="0.01"/>
+                                            <mass value="${m}"/>
                                             <!-- ORIGINAL value taken from Inertial_calculator.py -->
                                             <!-- <inertia ixx="2.56e-07" ixy="0.0" ixz="0.0" iyy="2.56e-07" iyz="0.0" izz="2.56e-07"/> -->
@@ -209,5 +245,5 @@
                                         </collision>
                                         <visual>
-                                            <origin xyz="0 0 0" rpy="0 0 0"/>
+                                            <xacro:visual_origin/>
                                             <geometry>
                                                 <sphere radius="0.008"/>
@@ -218,5 +254,5 @@
                                         <inertial>
                                             <origin xyz="0 0 0.01" rpy="0 0 0"/> <!--FOOT-->
-                                            <mass value="0.01"/>
+                                            <mass value="${m}"/>
                                             <!-- ORIGINAL value taken from Inertial_calculator.py -->
                                             <!-- <inertia ixx="2.56e-07" ixy="0.0" ixz="0.0" iyy="2.56e-07" iyz="0.0" izz="2.56e-07"/> -->
@@ -231,5 +267,5 @@
                                         </collision>
                                         <visual>
-                                            <origin xyz="0 0 0" rpy="0 0 0"/>
+                                            <xacro:visual_origin/>
                                             <geometry>
                                                 <sphere radius="0.008"/>
@@ -240,5 +276,5 @@
                                         <inertial>
                                             <origin xyz="0 0 0.01" rpy="0 0 0"/> <!--FOOT-->
-                                            <mass value="0.01"/>
+                                            <mass value="${m}"/>
                                             <!-- ORIGINAL value taken from Inertial_calculator.py -->
                                             <!-- <inertia ixx="2.56e-07" ixy="0.0" ixz="0.0" iyy="2.56e-07" iyz="0.0" izz="2.56e-07"/> -->
@@ -253,5 +289,5 @@
                                         </collision>
                                         <visual>
-                                            <origin xyz="0 0 0" rpy="0 0 0"/>
+                                            <xacro:visual_origin/>
                                             <geometry>
                                                 <sphere radius="0.008"/>
@@ -350,9 +386,4 @@
 <!-- ################### TRANSMISSION Definitions ############################# -->
 <!-- ################### TRANSMISSION Definitions ############################# -->
-    <gazebo>
-        <plugin name="gazebo_ros_control" filename="libgazebo_ros_control.so">
-            <robotNamespace>/gurdy</robotNamespace>
-        </plugin>
-    </gazebo>
             <transmission name="transmission_head_upperlegM1">
                 <type>transmission_interface/SimpleTransmission</type>
