Commit message: ofc it was 1 flippin typo that ruined everything. i wrote foot_M# instead of footM#...

File: my_gurdy_description/robots/gurdy.urdf (robot description, URDF)
Before this commit: robot gurdy, 11 links, 10 joints
Links:
- removed link foot_M1_link
- removed link foot_M2_link
- removed link foot_M3_link
- removed link lower_leg_M1_link
- removed link lower_leg_M2_link
- removed link lower_leg_M3_link
- removed link upper_leg_M1_link
- removed link upper_leg_M2_link
- removed link upper_leg_M3_link
- added link footM1_link, mass 0.01; collision sphere radius=0.008; visual sphere radius=0.008
- added link footM2_link, mass 0.01; collision sphere radius=0.008; visual sphere radius=0.008
- added link footM3_link, mass 0.01; collision sphere radius=0.008; visual sphere radius=0.008
- added link lowerleg_M1_link, mass 0.01; collision cylinder length=0.06 radius=0.0015; visual mesh filename=package://gurdy_description/models/gurdy/meshes/gurdy_lower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
- added link lowerleg_M2_link, mass 0.01; collision cylinder length=0.06 radius=0.0015; visual mesh filename=package://gurdy_description/models/gurdy/meshes/gurdy_lower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
- added link lowerleg_M3_link, mass 0.01; collision cylinder length=0.06 radius=0.0015; visual mesh filename=package://gurdy_description/models/gurdy/meshes/gurdy_lower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
- added link upperleg_M1_link, mass 0.01; collision cylinder length=0.06 radius=0.0025; visual mesh filename=package://gurdy_description/models/gurdy/meshes/gurdy_highe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
- added link upperleg_M2_link, mass 0.01; collision cylinder length=0.06 radius=0.0025; visual mesh filename=package://gurdy_description/models/gurdy/meshes/gurdy_highe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
- added link upperleg_M3_link, mass 0.01; collision cylinder length=0.06 radius=0.0025; visual mesh filename=package://gurdy_description/models/gurdy/meshes/gurdy_highe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
Joints:
- removed joint head_upper_legM1_joint
- removed joint head_upper_legM2_joint
- removed joint head_upper_legM3_joint
- removed joint upper_legM1_lowerlegM1_joint
- removed joint upper_legM2_lowerlegM2_joint
- removed joint upper_legM3_lowerlegM3_joint
- added joint head_upperlegM1_joint: type revolute, parent head_link, child upperleg_M1_link, origin xyz=-0.02165 -0.0125 -0.008 rpy=3.14159 0 0.523599, axis 0 1 0, limit lower=-1.57 upper=0.0 effort=1.0 velocity=0.005
- added joint head_upperlegM2_joint: type revolute, parent head_link, child upperleg_M2_link, origin xyz=0.02165 -0.0125 -0.008 rpy=3.14159 0 2.61799, axis 0 1 0, limit lower=-1.57 upper=0.0 effort=1.0 velocity=0.005
- added joint head_upperlegM3_joint: type revolute, parent head_link, child upperleg_M3_link, origin xyz=0 0.025 -0.008 rpy=3.14159 0 -1.5708, axis 0 1 0, limit lower=-1.57 upper=0.0 effort=1.0 velocity=0.005
- added joint upperlegM1_lowerlegM1_joint: type revolute, parent upperleg_M1_link, child lowerleg_M1_link, origin xyz=0 0.0095 0.06 rpy=0 0 3.14159, axis 0 1 0, limit lower=-2.65 upper=0 effort=1.0 velocity=0.005
- added joint upperlegM2_lowerlegM2_joint: type revolute, parent upperleg_M2_link, child lowerleg_M2_link, origin xyz=0 0.0095 0.06 rpy=0 0 3.14159, axis 0 1 0, limit lower=-2.65 upper=0 effort=1.0 velocity=0.005
- added joint upperlegM3_lowerlegM3_joint: type revolute, parent upperleg_M3_link, child lowerleg_M3_link, origin xyz=0 0.0095 0.06 rpy=0 0 3.14159, axis 0 1 0, limit lower=-2.65 upper=0 effort=1.0 velocity=0.005

File: my_gurdy_description/robots/gurdy.urdf.xacro (robot description, xacro)
@@ -6,6 +6,6 @@
 <!--base_link :         box size="0.01 0.01 0.01"                   mass=None, -->
 <!--head_link :         cylinder radius="0.05"      length="0.04"   mass value="0.01"-->
-<!--upper_leg_links :   cylinder radius="0.0025"    length="0.06"   mass value="0.01"-->
-<!--lower_leg_links :   cylinder radius="0.0015"    length="0.06"   mass value="0.01"-->
+<!--upperleg_links :   cylinder radius="0.0025"    length="0.06"   mass value="0.01"-->
+<!--lowerleg_links :   cylinder radius="0.0015"    length="0.06"   mass value="0.01"-->
 <!--foot_links :        sphere   radius="0.008"                     mass value="0.01"-->
 <!--Friction is vital in the foot links. Try different values and see the effect on locomotion. These are some orientative values:-->
@@ -28,12 +28,12 @@
 </gazebo>
 <!-- You can perform the basic operations (+,-,*,/), the unary minus, and use parenthesis. This allows you to, for example, calculate the inertias based on the dimensions directly in the XACRO file. -->
-<xacro:property name="head_ixx" value="${( (m/12.0) * (3*head_radius*head_radius + head_length*head_length) )}"/>
-<!-- Another example would be symmetrically-positioned links or joints. -->
-<xacro:property name="head_iyy" value="${head_ixx}"/>
-<xacro:property name="head_izz" value="( (m*head_radius*head_radius) / (2.0) )"/>
 <xacro:property name="m" value="0.01"/>
 <xacro:property name="head_radius" value="0.05"/>
 <xacro:property name="head_length" value="0.04"/>
 <xacro:property name="head_z_origin" value="0.02"/>
+<xacro:property name="head_ixx" value="${( (m/12.0) * (3*head_radius*head_radius + head_length*head_length) )}"/>
+<!-- Another example would be symmetrically-positioned links or joints. -->
+<xacro:property name="head_iyy" value="${head_ixx}"/>
+<xacro:property name="head_izz" value="${( (m*head_radius*head_radius) / (2.0) )}"/>
 <!-- MACROS
 This is by far the most useful feature of XACROS. There are two main types of MACROS: -->
@@ -46,10 +46,10 @@
 </xacro:macro>
 <!--######################## UPPER LEG ########################-->
-<xacro:property name="upper_leg_radius" value="0.0025"/>
-<xacro:property name="upper_leg_length" value="0.06"/>
-<xacro:macro name="upper_leg_origin">
+<xacro:property name="upperleg_radius" value="0.0025"/>
+<xacro:property name="upperleg_length" value="0.06"/>
+<xacro:macro name="upperleg_origin">
     <origin xyz="0 0 0.02" rpy="0 0 0"/> <!--UPPER-->
 </xacro:macro>
-<xacro:macro name="upper_leg_link_inertia">
+<xacro:macro name="upperleg_link_inertia">
     <!-- ORIGINAL value taken from Inertial_calculator.py -->
     <!-- <inertia ixx="3.015625e-06" ixy="0.0" ixz="0.0" iyy="3.015625e-06" iyz="0.0" izz="3.125e-08"/> -->
@@ -58,15 +58,15 @@
 </xacro:macro>
 <!-- PARAMETERISED MACRO -->
-<xacro:macro name="generate_upper_leg_link" params="num">
-    <link name="upper_leg_M${num}_link"><!--UPPER-->
+<xacro:macro name="generate_upperleg_link" params="num">
+    <link name="upperleg_M${num}_link"><!--UPPER-->
         <inertial>
-            <xacro:upper_leg_origin/>
+            <xacro:upperleg_origin/>
             <mass value="${m}"/>
-            <xacro:upper_leg_link_inertia/>
+            <xacro:upperleg_link_inertia/>
         </inertial>
         <collision>
-            <xacro:upper_leg_origin/>
-            <geometry>
-                <cylinder radius="${upper_leg_radius}" length="${upper_leg_length}"/>
+            <xacro:upperleg_origin/>
+            <geometry>
+                <cylinder radius="${upperleg_radius}" length="${upperleg_length}"/>
             </geometry>
         </collision>
@@ -80,10 +80,10 @@
 </xacro:macro>
 <!--######################## LOWER LEG ########################-->
-<xacro:property name="lower_leg_radius" value="0.0015"/>
-<xacro:property name="lower_leg_length" value="0.06"/>
-<xacro:macro name="lower_leg_origin">
+<xacro:property name="lowerleg_radius" value="0.0015"/>
+<xacro:property name="lowerleg_length" value="0.06"/>
+<xacro:macro name="lowerleg_origin">
     <origin xyz="0 0 0.03" rpy="0 0 0"/> <!--LOWER-->
 </xacro:macro>
-<xacro:macro name="lower_leg_link_inertia">
+<xacro:macro name="lowerleg_link_inertia">
     <!-- ORIGINAL value taken from Inertial_calculator.py -->
     <!-- <inertia ixx="3.005625e-06" ixy="0.0" ixz="0.0" iyy="3.005625e-06" iyz="0.0" izz="1.125e-08"/> -->
@@ -92,15 +92,15 @@
 </xacro:macro>
 <!-- PARAMETERISED MACRO -->
-<xacro:macro name="generate_lower_leg_link" params="num">
-    <link name="lower_leg_M${num}_link"><!--UPPER-->
+<xacro:macro name="generate_lowerleg_link" params="num">
+    <link name="lowerleg_M${num}_link"><!--UPPER-->
         <inertial>
-            <xacro:lower_leg_origin/>
+            <xacro:lowerleg_origin/>
             <mass value="${m}"/>
-            <xacro:lower_leg_link_inertia/>
+            <xacro:lowerleg_link_inertia/>
         </inertial>
         <collision>
-            <xacro:lower_leg_origin/>
-            <geometry>
-                <cylinder radius="${lower_leg_radius}" length="${lower_leg_length}"/>
+            <xacro:lowerleg_origin/>
+            <geometry>
+                <cylinder radius="${lowerleg_radius}" length="${lowerleg_length}"/>
             </geometry>
         </collision>
@@ -126,5 +126,5 @@
 <!-- PARAMETERISED MACRO -->
 <xacro:macro name="generate_foot_link" params="num">
-    <link name="foot_M${num}_link"><!--UPPER-->
+    <link name="footM${num}_link"><!--UPPER-->
         <inertial>
             <xacro:foot_origin/>
@@ -188,5 +188,5 @@
                     <mass value="${m}"/>
                     <!-- <inertia ixx="7.58333333333e-06" ixy="0.0" ixz="0.0" iyy="7.58333333333e-06" iyz="0.0" izz="1.25e-05"/> -->
-                    <inertia ixx="${head_ixx}" ixy="0.0" ixz="0.0" iyy="head_iyy" iyz="0.0" izz="head_izz"/>
+                    <inertia ixx="${head_ixx}" ixy="0.0" ixz="0.0" iyy="${head_iyy}" iyz="0.0" izz="${head_izz}"/>
                 </inertial>
                 <collision>
@@ -204,10 +204,10 @@
                 </visual>
             </link>
-                    <xacro:generate_upper_leg_link num="1" />
-                    <xacro:generate_upper_leg_link num="2" />
-                    <xacro:generate_upper_leg_link num="3" />
-                            <xacro:generate_lower_leg_link num="1" />
-                            <xacro:generate_lower_leg_link num="2" />
-                            <xacro:generate_lower_leg_link num="3" />
+                    <xacro:generate_upperleg_link num="1" />
+                    <xacro:generate_upperleg_link num="2" />
+                    <xacro:generate_upperleg_link num="3" />
+                            <xacro:generate_lowerleg_link num="1" />
+                            <xacro:generate_lowerleg_link num="2" />
+                            <xacro:generate_lowerleg_link num="3" />
                                     <xacro:generate_foot_link num="1" />
                                     <xacro:generate_foot_link num="2" />
@@ -226,7 +226,7 @@
         <!--<axis xyz="0 0 0"/>-->
     </joint>
-            <joint name="head_upper_legM1_joint" type="revolute">
+            <joint name="head_upperlegM1_joint" type="revolute">
                 <parent link="head_link"/>
-                <child link="upper_leg_M1_link"/>
+                <child link="upperleg_M1_link"/>
                 <!--this is the Pitch value from the urdf to graphiz map pdf-->
                 <!--<origin xyz="-0.02165 -0.0125 -0.008" rpy="3.14159 -1.05879e-22 0.523599"/>-->
@@ -238,7 +238,7 @@
                 <axis xyz="0 1 0"/>
             </joint>
-            <joint name="head_upper_legM2_joint" type="revolute">
+            <joint name="head_upperlegM2_joint" type="revolute">
                 <parent link="head_link"/>
-                <child link="upper_leg_M2_link"/>
+                <child link="upperleg_M2_link"/>
                 <origin xyz="0.02165 -0.0125 -0.008" rpy="3.14159 0 2.61799"/>
                 <!--Rest NOT NEEDED for FIXED joint-->
@@ -246,7 +246,7 @@
                 <axis xyz="0 1 0"/>
             </joint>
-            <joint name="head_upper_legM3_joint" type="revolute">
+            <joint name="head_upperlegM3_joint" type="revolute">
                 <parent link="head_link"/>
-                <child link="upper_leg_M3_link"/>
+                <child link="upperleg_M3_link"/>
                 <origin xyz="0 0.025 -0.008" rpy="3.14159 0 -1.5708"/>
                 <!--Rest NOT NEEDED for FIXED joint-->
@@ -254,6 +254,6 @@
                 <axis xyz="0 1 0"/>
             </joint>
-                    <joint name="upper_legM1_lowerlegM1_joint" type="revolute">
-                        <parent link="upper_leg_M1_link"/>
+                    <joint name="upperlegM1_lowerlegM1_joint" type="revolute">
+                        <parent link="upperleg_M1_link"/>
                         <child link="lowerleg_M1_link"/>
                         <origin xyz="0 0.0095 0.06" rpy="0 0 3.14159"/>
@@ -261,6 +261,6 @@
                         <axis xyz="0 1 0"/>
                     </joint>
-                    <joint name="upper_legM2_lowerlegM2_joint" type="revolute">
-                        <parent link="upper_leg_M2_link"/>
+                    <joint name="upperlegM2_lowerlegM2_joint" type="revolute">
+                        <parent link="upperleg_M2_link"/>
                         <child link="lowerleg_M2_link"/>
                         <origin xyz="0 0.0095 0.06" rpy="0 0 3.14159"/>
@@ -268,6 +268,6 @@
                         <axis xyz="0 1 0"/>
                     </joint>
-                    <joint name="upper_legM3_lowerlegM3_joint" type="revolute">
-                        <parent link="upper_leg_M3_link"/>
+                    <joint name="upperlegM3_lowerlegM3_joint" type="revolute">
+                        <parent link="upperleg_M3_link"/>
                         <child link="lowerleg_M3_link"/>
                         <origin xyz="0 0.0095 0.06" rpy="0 0 3.14159"/>
@@ -304,64 +304,64 @@
 <!-- ################### TRANSMISSION Definitions ############################# -->
 <!-- ################### TRANSMISSION Definitions ############################# -->
-            <transmission name="transmission_head_upper_legM1">
+            <!-- <transmission name="transmission_head_upperlegM1">
                 <type>transmission_interface/SimpleTransmission</type>
-                <joint name="head_upper_legM1_joint">
+                <joint name="head_upperlegM1_joint">
                     <hardwareInterface>EffortJointInterface</hardwareInterface>
                 </joint>
-                <actuator name="motor_head_upper_legM1">
+                <actuator name="motor_head_upperlegM1">
                     <hardwareInterface>EffortJointInterface</hardwareInterface>
                     <mechanicalReduction>1</mechanicalReduction>
                 </actuator>
             </transmission>
-            <transmission name="transmission_head_upper_legM2">
+            <transmission name="transmission_head_upperlegM2">
                 <type>transmission_interface/SimpleTransmission</type>
-                <joint name="head_upper_legM2_joint">
+                <joint name="head_upperlegM2_joint">
                     <hardwareInterface>EffortJointInterface</hardwareInterface>
                 </joint>
-                <actuator name="motor_head_upper_legM2">
+                <actuator name="motor_head_upperlegM2">
                     <hardwareInterface>EffortJointInterface</hardwareInterface>
                     <mechanicalReduction>1</mechanicalReduction>
                 </actuator>
             </transmission>
-            <transmission name="transmission_head_upper_legM3">
+            <transmission name="transmission_head_upperlegM3">
                 <type>transmission_interface/SimpleTransmission</type>
-                <joint name="head_upper_legM3_joint">
+                <joint name="head_upperlegM3_joint">
                     <hardwareInterface>EffortJointInterface</hardwareInterface>
                 </joint>
-                <actuator name="motor_head_upper_legM3">
+                <actuator name="motor_head_upperlegM3">
                     <hardwareInterface>EffortJointInterface</hardwareInterface>
                     <mechanicalReduction>1</mechanicalReduction>
                 </actuator>
             </transmission>
-                    <transmission name="transmission_upper_legM1_lowerlegM1">
+                    <transmission name="transmission_upperlegM1_lowerlegM1">
                         <type>transmission_interface/SimpleTransmission</type>
-                        <joint name="upper_legM1_lowerlegM1_joint">
+                        <joint name="upperlegM1_lowerlegM1_joint">
                             <hardwareInterface>EffortJointInterface</hardwareInterface>
                         </joint>
-                        <actuator name="motor_upper_legM1_lowerlegM1">
+                        <actuator name="motor_upperlegM1_lowerlegM1">
                             <hardwareInterface>EffortJointInterface</hardwareInterface>
                             <mechanicalReduction>1</mechanicalReduction>
                         </actuator>
                     </transmission>
-                    <transmission name="transmission_upper_legM2_lowerlegM2">
+                    <transmission name="transmission_upperlegM2_lowerlegM2">
                         <type>transmission_interface/SimpleTransmission</type>
-                        <joint name="upper_legM2_lowerlegM2_joint">
+                        <joint name="upperlegM2_lowerlegM2_joint">
                             <hardwareInterface>EffortJointInterface</hardwareInterface>
                         </joint>
-                        <actuator name="motor_upper_legM2_lowerlegM2">
+                        <actuator name="motor_upperlegM2_lowerlegM2">
                             <hardwareInterface>EffortJointInterface</hardwareInterface>
                             <mechanicalReduction>1</mechanicalReduction>
                         </actuator>
                     </transmission>
-                    <transmission name="transmission_upper_legM3_lowerlegM3">
+                    <transmission name="transmission_upperlegM3_lowerlegM3">
                         <type>transmission_interface/SimpleTransmission</type>
-                        <joint name="upper_legM3_lowerlegM3_joint">
+                        <joint name="upperlegM3_lowerlegM3_joint">
                             <hardwareInterface>EffortJointInterface</hardwareInterface>
                         </joint>
-                        <actuator name="motor_upper_legM3_lowerlegM3">
+                        <actuator name="motor_upperlegM3_lowerlegM3">
                             <hardwareInterface>EffortJointInterface</hardwareInterface>
                             <mechanicalReduction>1</mechanicalReduction>
                         </actuator>
-                    </transmission>
+                    </transmission> -->
 <!-- ################### MATERIALS Definitions ############################# -->
 <!-- ################### MATERIALS Definitions ############################# -->
@@ -408,5 +408,5 @@
 <!-- ################### SENSOR Definitions ############################# -->
 <!-- ################### SENSOR Definitions ############################# -->
-    <gazebo>
+    <!-- <gazebo>
         <plugin name="gazebo_ros_imu_controller" filename="libgazebo_ros_imu.so">
             <robotNamespace>/gurdy</robotNamespace>
@@ -420,4 +420,4 @@
             <gaussianNoise>0</gaussianNoise>
         </plugin>
-</gazebo>
+</gazebo> -->
 </robot>
