Commit message: tidied up urdf with xacro, so im mostly done with this project. next is to make code notes with all the rviz, gazebo and rqt tools i used for future ref

File: my_gurdy_description/urdf/gurdy.urdf (robot description, URDF)
Before this commit: robot gurdy, 11 links, 10 joints
Links:
- removed link lowerleg_M1_link
- removed link lowerleg_M2_link
- removed link lowerleg_M3_link
- removed link upperleg_M1_link
- removed link upperleg_M2_link
- removed link upperleg_M3_link
- added link lowerlegM1_link, mass 0.01; collision cylinder length=0.06 radius=0.0015; visual mesh filename=package://gurdy_description/models/gurdy/meshes/gurdy_lower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
- added link lowerlegM2_link, mass 0.01; collision cylinder length=0.06 radius=0.0015; visual mesh filename=package://gurdy_description/models/gurdy/meshes/gurdy_lower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
- added link lowerlegM3_link, mass 0.01; collision cylinder length=0.06 radius=0.0015; visual mesh filename=package://gurdy_description/models/gurdy/meshes/gurdy_lower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
- added link upperlegM1_link, mass 0.01; collision cylinder length=0.06 radius=0.0025; visual mesh filename=package://gurdy_description/models/gurdy/meshes/gurdy_highe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
- added link upperlegM2_link, mass 0.01; collision cylinder length=0.06 radius=0.0025; visual mesh filename=package://gurdy_description/models/gurdy/meshes/gurdy_highe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
- added link upperlegM3_link, mass 0.01; collision cylinder length=0.06 radius=0.0025; visual mesh filename=package://gurdy_description/models/gurdy/meshes/gurdy_highe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
Joints:
- removed joint basefoot_peg_M1_basefoot_peg_M1_joint_joint
- removed joint basefoot_peg_M2_basefoot_peg_M2_joint_joint
- removed joint basefoot_peg_M3_basefoot_peg_M3_joint_joint
- added joint lowerlegM1_footM1_joint: type fixed, parent lowerlegM1_link, child footM1_link, origin xyz=0 0 0.06 rpy=0 0 0
- added joint lowerlegM2_footM2_joint: type fixed, parent lowerlegM2_link, child footM2_link, origin xyz=0 0 0.06 rpy=0 0 0
- added joint lowerlegM3_footM3_joint: type fixed, parent lowerlegM3_link, child footM3_link, origin xyz=0 0 0.06 rpy=0 0 0
- joint head_upperlegM1_joint: child upperleg_M1_link -> upperlegM1_link
- joint head_upperlegM2_joint: child upperleg_M2_link -> upperlegM2_link
- joint head_upperlegM3_joint: child upperleg_M3_link -> upperlegM3_link
- joint upperlegM1_lowerlegM1_joint: child lowerleg_M1_link -> lowerlegM1_link; parent upperleg_M1_link -> upperlegM1_link
- joint upperlegM2_lowerlegM2_joint: child lowerleg_M2_link -> lowerlegM2_link; parent upperleg_M2_link -> upperlegM2_link
- joint upperlegM3_lowerlegM3_joint: child lowerleg_M3_link -> lowerlegM3_link; parent upperleg_M3_link -> upperlegM3_link
